Commit message: uploading code for final project

File: rotors_description/urdf/firefly.xacro (robot description, xacro)
@@ -199,5 +199,5 @@
     <joint name="camera_joint" type="fixed">
     <axis xyz="0 1 0" />
-    <origin xyz="-0.1 0 0" rpy="0 0 0"/>
+    <origin xyz="-0.1 0 0.0" rpy="0 0 0"/>
     <parent link="${namespace}/base_link"/>
     <child link="marker"/>

File: rotors_description/urdf/firefly2.xacro (robot description, xacro)
@@ -198,5 +198,5 @@
     <joint name="camera_joint" type="fixed">
     <axis xyz="0 1 0" />
-    <origin xyz="0.1 0 0.2" rpy="0 0 0"/>
+    <origin xyz="0.1 0 0.21" rpy="0 0 0"/>
     <parent link="${namespace}/base_link"/>
     <child link="camera_link"/>
